Commit message: added cube object for debugging

File: roboverse/envs/assets/objects/bowl.urdf (robot description, URDF)
Before this commit: robot bowl.urdf, 5 links, 4 joints
Links:
- removed link handle_m
- link base: geometry collision box size=.1 1.1 .5; collision box size=.1 1.1 .5
- link handle: mass None -> .001; geometry collision box size=0.5 0.2 .2; visual box size=0.5 0.2 .2
Joints:
- removed joint j_handle_m

Commit message: added bbox debug drawing

File: roboverse/envs/assets/objects/bowl.urdf (robot description, URDF)
Before this commit: robot bowl.urdf, 4 links, 3 joints
Links:
- link handle: mass .001 -> .1
- link lid: mass .001 -> .1

Commit message: new objects; rendering

File: roboverse/envs/assets/objects/bowl.urdf (robot description, URDF)
Before this commit: robot bowl.urdf, 4 links, 3 joints
Links:
- link lid: mass .1 -> .25
Joints:
- removed joint j_base
- removed joint j_handle
- removed joint j_lid
- added joint base_joint: type fixed, parent world, child base
- added joint handle_joint: type fixed, parent lid, child handle, origin xyz=0 0 0.1 rpy=0 0 0
- added joint lid_joint: type prismatic, parent base, child lid, origin xyz=0 0 0.35 rpy=0 0 0, axis 0 1 0, limit lower=0 upper=1 effort=100 velocity=100

File: roboverse/envs/assets/objects/cube.urdf (robot description, URDF)
Before this commit: robot sphere.urdf, 1 links, 0 joints
Links:
- removed link sphere
- added link cube, mass 1; collision box size=1 1 1; visual box size=1 1 1

Commit message: fixed spam

File: roboverse/envs/assets/objects/bowl.urdf (robot description, URDF)
Before this commit: robot bowl.urdf, 4 links, 3 joints
Links:
- link base: geometry collision box size=.05 1 .5; collision box size=.05 1 .5

File: roboverse/envs/assets/objects/spam/spam.urdf (robot description, URDF)
Before this commit: robot spam.urdf, 1 links, 0 joints
Links:
- link spam: mass .1 -> .25; geometry collision box size=1.75 1.75 1.75; visual mesh filename=roboverse/envs/assets/objects/spam/spam.obj scale=1 1 1
