Commit message: added auto env registration, cleaned spam env

File: roboverse/envs/assets/objects/spam/spam.urdf (robot description, URDF)
Before this commit: robot spam.urdf, 1 links, 0 joints
Links:
- link spam: geometry collision box size=1.95 1.95 1.95; visual mesh filename=roboverse/envs/assets/objects/spam/spam.obj scale=1 1 1

Commit message: added noisy grasping policy

File: roboverse/envs/assets/objects/spam/spam.urdf (robot description, URDF)
Before this commit: robot spam.urdf, 1 links, 0 joints
Links:
- link spam: mass .25 -> .5
