Commit message: Change widow URDF to make more realistic

File: roboverse/envs/assets/widowx/widowx1.urdf (robot description, URDF)
Before this commit: robot widowx, 10 links, 9 joints
Joints:
- joint gripper_prismatic_joint_2: axis 0 -1 0 -> 0 1 0; origin xyz=0 0.027 0 rpy=0 0 0 -> xyz=0 0 0 rpy=0 0 0
- joint joint_1: limit effort=0 velocity=0.785 -> lower=-2.617 upper=2.617 effort=0 velocity=0.785; origin xyz=0 0 -0.125 rpy=0 3.14159 0 -> xyz=0 0 0.125 rpy=0 0 0
- joint joint_2: limit lower=-1.571 upper=0 effort=0 velocity=1.571 -> lower=-1.571 upper=1.571 effort=0 velocity=1.571
