Commit message: Add general robot base env (shouldn't be instantiated)

File: roboverse/envs/assets/widowx/widowx.urdf (robot description, URDF)
Before this commit: robot widowx, 10 links, 9 joints
Joints:
- joint gripper_prismatic_joint_2: axis 0 1 0 -> 0 -1 0; origin xyz=0 0 0 rpy=0 0 0 -> xyz=0 0.027 0 rpy=0 0 0

Commit message: Edit urdf, add downwards and upwards configurations, add rotation to scripted grasping

File: roboverse/envs/assets/widowx/widowx.urdf (robot description, URDF)
Before this commit: robot widowx, 10 links, 9 joints
Joints:
- joint joint_1: origin xyz=0 0 -0.125 rpy=0 3.14159 0 -> xyz=0 0 0.125 rpy=0 0 0
- joint joint_2: limit lower=-1.571 upper=0 effort=0 velocity=1.571 -> lower=-1.571 upper=1.571 effort=0 velocity=1.571
- joint joint_4: limit lower=-1.745 upper=1.745 effort=0 velocity=1.571 -> lower=-2.745 upper=2.745 effort=0 velocity=1.571

File: roboverse/envs/assets/widowx/widowxdownwards.urdf (robot description, URDF)
Before this commit: robot widowx, 10 links, 9 joints
Joints:
- joint gripper_prismatic_joint_2: axis 0 1 0 -> 0 -1 0; origin xyz=0 0 0 rpy=0 0 0 -> xyz=0 0.027 0 rpy=0 0 0
- joint joint_1: limit lower=-2.617 upper=2.617 effort=0 velocity=0.785 -> effort=0 velocity=0.785; origin xyz=0 0 0.125 rpy=0 0 0 -> xyz=0 0 -0.125 rpy=0 3.14159 0
- joint joint_2: limit lower=-1.571 upper=1.571 effort=0 velocity=1.571 -> lower=-1.571 upper=0 effort=0 velocity=1.571
- joint joint_4: limit lower=-1.745 upper=1.745 effort=0 velocity=1.571 -> lower=-2.745 upper=2.745 effort=0 velocity=1.571
