Commit message: Unrobust but working box packing.

File: roboverse/envs/assets/objects/box/box.urdf (robot description, URDF)
Before this commit: robot bowl.urdf, 4 links, 3 joints
Links:
- removed link handle
- added link handle_r, mass .1; collision cylinder length=0.6 radius=0.05; visual cylinder length=0.6 radius=0.05
- link base: geometry collision box size=.05 1 .5; collision box size=.05 1 .5
Joints:
- removed joint handle_joint
- added joint handle_r_joint: type fixed, parent lid, child handle_r, origin xyz=-0.8 0 -0.1 rpy=0 0 0
- joint lid_joint: axis 0 1 0 -> 1 0 0; limit lower=0 upper=2 effort=100 velocity=100 -> lower=-3 upper=0 effort=100 velocity=100; origin xyz=0.5 0 0.3 rpy=0 0 0 -> xyz=0.5 0.5 0.3 rpy=0 0 0

File: roboverse/envs/assets/objects/hinge/hinge.urdf (robot description, URDF)
Before this commit: robot bowl.urdf, 4 links, 3 joints
Joints:
- joint lid_joint: limit lower=0 upper=1 effort=100 velocity=100 -> lower=0 upper=1 effort=50 velocity=50
