Commit message: made gripper heavier; reduced gripper velocity multiplier in ik

File: roboverse/envs/assets/sawyer_robot/sawyer_description/urdf/sawyer_xacro.urdf (robot description, URDF)
Before this commit: robot sawyer, 26 links, 25 joints
Links:
- link right_gripper_l_finger: mass 0.001 -> 0.1
- link right_gripper_r_finger: mass 0.001 -> 0.1

Commit message: added gripper site

File: roboverse/envs/assets/sawyer_robot/sawyer_description/urdf/sawyer_xacro.urdf (robot description, URDF)
Before this commit: robot sawyer, 26 links, 25 joints
Links:
- added link gripper_site; visual box size=.01 .01 .01
Joints:
- added joint right_electric_gripper_base: type fixed, parent right_electric_gripper_base, child gripper_site, origin xyz=0 0 0.1 rpy=0 0 0

Commit message: added default inertia info to urdf

File: roboverse/envs/assets/sawyer_robot/sawyer_description/urdf/sawyer_xacro.urdf (robot description, URDF)
Before this commit: robot sawyer, 27 links, 26 joints
Links:
- link gripper_site: mass None -> 1
- link head_camera: mass None -> 1
- link right_hand_camera: mass None -> 1
- link right_wrist: mass None -> 1

Commit message: Make gripper wider

File: roboverse/envs/assets/sawyer_robot/sawyer_description/urdf/sawyer_xacro.urdf (robot description, URDF)
Before this commit: robot sawyer, 27 links, 26 joints
Joints:
- joint right_gripper_l_finger_joint: limit lower=0.0 upper=0.03 effort=20.0 velocity=5.0 -> lower=0.0 upper=0.05 effort=20.0 velocity=5.0
- joint right_gripper_r_finger_joint: limit lower=-0.045 upper=0.0 effort=20.0 velocity=5.0 -> lower=-0.065 upper=0.0 effort=20.0 velocity=5.0

Commit message: WIP

File: roboverse/envs/assets/sawyer_robot/sawyer_description/urdf/sawyer_xacro.urdf (robot description, URDF)
Before this commit: robot sawyer, 27 links, 26 joints
Joints:
- joint right_gripper_l_finger_joint: limit lower=0.0 upper=0.05 effort=20.0 velocity=5.0 -> lower=0.0 upper=0.03 effort=20.0 velocity=5.0
- joint right_gripper_r_finger_joint: limit lower=-0.065 upper=0.0 effort=20.0 velocity=5.0 -> lower=-0.045 upper=0.0 effort=20.0 velocity=5.0
