Commit message: cleaned up objects

File: roboverse/envs/assets/objects/bowl/bowl.urdf (robot description, URDF)
Before this commit: robot bowl.urdf, 4 links, 3 joints
Links:
- link base: geometry collision box size=.05 1 .5; collision box size=.05 1 .5

Commit message: lid on bowl is now free joint

File: roboverse/envs/assets/objects/bowl/bowl.urdf (robot description, URDF)
Before this commit: robot bowl.urdf, 4 links, 3 joints
Links:
- removed link handle
- removed link lid
- link base: geometry collision box size=.05 1 .6; collision box size=.05 1 .6
Joints:
- removed joint handle_joint
- removed joint lid_joint

Commit message: Different bowl shape

File: roboverse/envs/assets/objects/bowl/bowl.urdf (robot description, URDF)
Before this commit: robot bowl.urdf, 2 links, 1 joints
Links:
- link base: geometry collision box size=.05 1 .6; collision box size=.05 1 .6

File: roboverse/envs/assets/objects/bowl/lid.urdf (robot description, URDF)
Before this commit: robot bowl.urdf, 2 links, 1 joints
Links:
- link handle: mass .1 -> 1; geometry collision box size=0.5 0.1 .3; visual box size=0.5 0.1 .3
- link lid: mass .1 -> 1; geometry collision box size=1.05 1.05 .1; visual box size=1.05 1.05 .1
