Commit message: Functional Widow200 in sim with box-opening scripted policy. Add plotting functionality to widow box packing scripted policy. URDF friction changes to robot gripper and box handle. Functional Widow200 grasp environment with step and reset.

File: roboverse/envs/assets/interbotix_descriptions/urdf/wx200.urdf (robot description, URDF)
Before this commit: robot wx200, 13 links, 12 joints
Links:
- link wx200/base_link: mass 0.540142 -> 0
Joints:
- joint wrist_rotate: origin xyz=0.065 0 0 rpy=-3.141592653589793 0 0 -> xyz=0.065 0 0 rpy=1.57 0 0
