Commit message: Revert "Mostly working widow250s env."
This reverts commit 88e20897a61d76d78ad4c40d313903b4fc08a1fb.

File: roboverse/envs/assets/interbotix_descriptions/urdf/wx250s.urdf (robot description, URDF)
Before this commit: robot wx250s, 14 links, 13 joints
Links:
- link /base_link: mass 0.0 -> 0.538736

Commit message: finished bridge envs

File: roboverse/envs/assets/interbotix_descriptions/urdf/wx250s.urdf (robot description, URDF)
Before this commit: robot wx250s, 14 links, 13 joints
Joints:
- joint right_finger: limit lower=-0.037 upper=-0.015 effort=10 velocity=1 -> lower=-0.037 upper=-0.05 effort=10 velocity=1
