Commit message: ckpt1: slanted walls, breset-free sliding, drawer re-adjustment

File: roboverse/envs/assets/bullet-objects/drawer/drawer_lightblue_base_longhandle_rgba.urdf (robot description, URDF)
Before this commit: robot bowl.urdf, 6 links, 5 joints
Joints:
- joint base_frame_joint: limit lower=-1.25 upper=0 effort=100 velocity=100 -> lower=-.95 upper=-.15 effort=100 velocity=100

File: roboverse/envs/assets/bullet-objects/wall/wall_narrow_r.urdf (robot description, URDF)
Before this commit: robot bowl.urdf, 2 links, 1 joints
Links:
- link base: geometry collision box size=.01 .65 .2; collision box size=.01 1 .2

Commit message: ckpt7: data collection with new env

File: roboverse/envs/assets/bullet-objects/drawer/drawer_lightblue_base_longhandle_rgba.urdf (robot description, URDF)
Before this commit: robot bowl.urdf, 6 links, 5 joints
Joints:
- joint base_frame_joint: limit lower=-.95 upper=-.15 effort=100 velocity=100 -> lower=-1.25 upper=0 effort=100 velocity=100
